Commit message: Using ORB SLAM 2 for webcam

File: src/rob_description/urdf/spider_assembly.xacro (robot description, xacro)
@@ -603,5 +603,5 @@
     <origin xyz="-0.02 -0.002 0.023" rpy="0 0 0" />
   </joint>
-  <link name="ultrasonic_link">
+  <link name="sonar_link">
     <collision>
       <geometry>
@@ -620,5 +620,5 @@
   <joint name="ultrasonic_sensor_joint" type="fixed">
     <parent link="base_link"/>
-    <child link="ultrasonic_link"/>
+    <child link="sonar_link"/>
     <origin xyz="0.01 -0.002 0.1" rpy="0 0 0"/>
   </joint>

Commit message: Robot urdf files with gazebo plugins

File: src/rob_description/urdf/spider_assembly.xacro (robot description, xacro)
@@ -434,5 +434,5 @@
     <child link="waist_link" />
     <axis xyz="0 0 1" />
-    <limit lower="-1" upper="2.14" effort="1" velocity="0.524" />
+    <limit lower="-0.6" upper="2.7302" effort="1" velocity="0.524" />
   </joint>
   <link name="shoulder_link">
@@ -621,5 +621,5 @@
     <parent link="base_link"/>
     <child link="sonar_link"/>
-    <origin xyz="0.01 -0.002 0.1" rpy="0 0 0"/>
+    <origin xyz="0.01 -0.002 10" rpy="0 0 0"/>
   </joint>
   <transmission name="waist_link">

File: src/rob_description/urdf/spider_assembly_urdf.urdf (robot description, URDF)
Before this commit: robot rob_description, 21 links, 20 joints
Joints:
- joint waist_joint: limit lower=-0.6 upper=2.54 effort=5 velocity=3 -> lower=-0.6 upper=2.7302 effort=5 velocity=3
