Commit message: MoveIt planning launch files

File: src/moveit_robot_sim/config/gazebo_rob_description.urdf (robot description, URDF)
Before this commit: robot rob_description, 21 links, 20 joints
Joints:
- joint elbow_joint: limit lower=-1.8 upper=1.34 effort=75 velocity=3 -> lower=-1.8 upper=1.34 effort=5 velocity=3
- joint gripper_joint: limit lower=-1.1 upper=-0.4 effort=75 velocity=3 -> lower=-1.1 upper=-0.4 effort=5 velocity=3
- joint leg_1_1_joint: limit lower=-1.3 upper=1.3 effort=75 velocity=3 -> lower=-1.3 upper=1.3 effort=5 velocity=3
- joint leg_1_2_joint: limit lower=-1.57 upper=1.57 effort=75 velocity=3 -> lower=-1.57 upper=1.57 effort=5 velocity=3
- joint leg_1_3_joint: limit lower=-3.09 upper=0.5 effort=75 velocity=3 -> lower=-3.09 upper=0.5 effort=5 velocity=3
- joint leg_2_1_joint: limit lower=-1.3 upper=1.3 effort=75 velocity=3 -> lower=-1.3 upper=1.3 effort=5 velocity=3
- joint leg_2_2_joint: limit lower=-1.57 upper=1.57 effort=75 velocity=3 -> lower=-1.57 upper=1.57 effort=5 velocity=3
- joint leg_2_3_joint: limit lower=-3.09 upper=0.5 effort=75 velocity=3 -> lower=-3.09 upper=0.5 effort=5 velocity=3
- joint leg_3_1_joint: limit lower=-1.3 upper=1.3 effort=75 velocity=3 -> lower=-1.3 upper=1.3 effort=5 velocity=3
- joint leg_3_2_joint: limit lower=-1.57 upper=1.57 effort=75 velocity=3 -> lower=-1.57 upper=1.57 effort=5 velocity=3
- joint leg_3_3_joint: limit lower=-3.09 upper=0.5 effort=75 velocity=3 -> lower=-3.09 upper=0.5 effort=5 velocity=3
- joint leg_4_1_joint: limit lower=-1.3 upper=1.3 effort=75 velocity=3 -> lower=-1.3 upper=1.3 effort=5 velocity=3
- joint leg_4_2_joint: limit lower=-1.57 upper=1.57 effort=75 velocity=3 -> lower=-1.57 upper=1.57 effort=5 velocity=3
- joint leg_4_3_joint: limit lower=-3.09 upper=0.5 effort=75 velocity=3 -> lower=-3.09 upper=0.5 effort=5 velocity=3
- joint shoulder_joint: limit lower=-2.04 upper=1.1 effort=75 velocity=3 -> lower=-2.04 upper=1.1 effort=5 velocity=3
- joint waist_joint: limit lower=-0.6 upper=2.54 effort=75 velocity=3 -> lower=-0.6 upper=2.54 effort=5 velocity=3
- joint wrist_joint: limit lower=0 upper=3.14 effort=75 velocity=3 -> lower=0 upper=3.14 effort=5 velocity=3
- joint wrist_pitch_joint: limit lower=-1.14 upper=2 effort=75 velocity=3 -> lower=-1.14 upper=2 effort=5 velocity=3
